File: PCB/tamagotchi.kicad_pcb (KiCad board)
At the start: 2 copper layers, 70.6 x 76 mm, 11 parts, among them SW1 SW_Push, SW2 SW_Push, SW3 SW_Push, U1 XIAO-ESP32-C3-SMD, U2 HS96L03W2C03

Commit message: Add files via upload
Parts:
- BT1, D1, D2, R1, R2: moved to B.Cu
- moved R2 7.83 mm to (173.6, 75.9), turned to 180 degrees
- moved R1 7.77 mm to (131.1, 76.3), turned to 180 degrees
- moved BT1 2.53 mm to (150.8, 65.2)
- turned D1 to 180 degrees
- turned D2 to 180 degrees
Routing:
- net Net-(U1-GPIO8_D8_SCK): track 44.1 -> 53.2 mm
- net Net-(D2-A): track 11.5 -> 6.41 mm
- net Net-(D1-A): track 7.17 -> 11.8 mm
- net Net-(U1-GPIO20_D7_RX): track 51.9 -> 55.9 mm
